File: Calculator.kicad_sch (KiCad schematic)
At the start: 55 parts, among them J1 Conn_01x02_Pin, J2 Conn_01x04, J3 DEM 128064E1 FGH, SW1 SW_Push, SW10 SW_Push, SW11 SW_Push, SW12 SW_Push, SW13 SW_Push, SW14 SW_Push, SW15 SW_Push, SW16 SW_Push, SW17 SW_Push, SW18 SW_Push, SW19 SW_Push, SW2 SW_Push, SW20 SW_Push, SW21 SW_Push, SW22 SW_Push, SW23 SW_Push, SW24 SW_Push, SW25 SW_Push, SW26 SW_Push, SW27 SW_Push, SW28 SW_Push, SW29 SW_Push, SW3 SW_Push, SW30 SW_Push, SW31 SW_Push, SW4 SW_Push, SW5 SW_Push, SW6 SW_Push, SW7 SW_Push, SW8 SW_Push, SW9 SW_Push, U1 STM32L071RZTx

Commit message: Update.
Connections:
- net A0: now also U1.2 (PC13)
- net C86: now also U1.21 (PA5)
- net LCD_RST: now also U1.5 (PH0)
- net NCS: now also U1.6 (PH1)
- net RD: now also U1.4 (PC15)
- net WR: now also U1.3 (PC14)
Other:
- moved on the sheet: C1, R1, R2, SW31
