File: KS100.kicad_pcb (KiCad board)
At the start: 2 copper layers, 80 x 80 mm, 55 parts, among them J1 Conn_01x02_Pin, J2 Conn_01x04, J3 DEM 128064E1 FGH, SW1 SW_Push, SW10 SW_Push, SW11 SW_Push, SW12 SW_Push, SW13 SW_Push, SW14 SW_Push, SW15 SW_Push, SW16 SW_Push, SW17 SW_Push, SW18 SW_Push, SW19 SW_Push, SW2 SW_Push, SW20 SW_Push, SW21 SW_Push, SW22 SW_Push, SW23 SW_Push, SW24 SW_Push, SW25 SW_Push, SW26 SW_Push, SW27 SW_Push, SW28 SW_Push, SW29 SW_Push, SW3 SW_Push, SW30 SW_Push, SW31 SW_Push, SW4 SW_Push, SW5 SW_Push, SW6 SW_Push, SW7 SW_Push, SW8 SW_Push, SW9 SW_Push, U1 STM32L071RZTx

Commit message: Update.
Connections:
- U1 pad 2: unconnected-(U1-PC13-Pad2) -> /Calculator/A0
- U1 pad 21: unconnected-(U1-PA5-Pad21) -> /Calculator/C86
- U1 pad 3: unconnected-(U1-PC14-Pad3) -> /Calculator/WR
- U1 pad 4: unconnected-(U1-PC15-Pad4) -> /Calculator/RD
- U1 pad 5: unconnected-(U1-PH0-Pad5) -> /Calculator/LCD_RST
- U1 pad 6: unconnected-(U1-PH1-Pad6) -> /Calculator/NCS
Routing:
- net /Calculator/C86: track 0.00 -> 33.1 mm, vias 0 -> 2
- net /Calculator/NCS: track 21.1 -> 41.8 mm, vias 1 -> 2
- net /Calculator/RD: track 21.1 -> 35.0 mm, vias 1 -> 2
- net /Calculator/WR: track 19.7 -> 32.3 mm, vias 1 -> 2
- net /Calculator/LCD_RST: track 20.1 -> 32.1 mm, vias 1 -> 2
- net /Calculator/A0: track 19.7 -> 30.4 mm, vias 1 -> 2
- net unconnected-(U1-PA2-Pad16): track 0.00 -> 2.13 mm, vias 0 -> 1
- net /Calculator/SI: track 24.6 -> 23.8 mm
