File: 01_EDA/Calculator.kicad_sch (KiCad schematic)
At the start: 55 parts, among them J1 Conn_01x02_Pin, J2 Conn_01x04, J3 DEM 128064E1 FGH, SW1 SW_Push, SW10 SW_Push, SW11 SW_Push, SW12 SW_Push, SW13 SW_Push, SW14 SW_Push, SW15 SW_Push, SW16 SW_Push, SW17 SW_Push, SW18 SW_Push, SW19 SW_Push, SW2 SW_Push, SW20 SW_Push, SW21 SW_Push, SW22 SW_Push, SW23 SW_Push, SW24 SW_Push, SW25 SW_Push, SW26 SW_Push, SW27 SW_Push, SW28 SW_Push, SW29 SW_Push, SW3 SW_Push, SW30 SW_Push, SW31 SW_Push, SW4 SW_Push, SW5 SW_Push, SW6 SW_Push, SW7 SW_Push, SW8 SW_Push, SW9 SW_Push, U1 STM32L071RZTx

Commit message: Update.
Parts:
- removed R10, R11, R12, R8: R_US, Resistor_SMD:R_0603_1608Metric_Pad0.98x0.95mm_HandSolder, symbol Device:R_US
- added R3, R4, R7: 1K, Resistor_SMD:R_0603_1608Metric_Pad0.98x0.95mm_HandSolder, symbol Device:R_US
- R1: now left out of the parts list
- R5, R6, R9: value R_US -> 1K
- R8: renamed from R7; value R_US -> 1K
- renumbered C7 to C10, C8 to C7, C9 to C8, C10 to C9, SW31 to SW21, SW21 to SW22, SW22 to SW23, SW23 to SW24, SW24 to SW25, SW25 to SW26, SW26 to SW27, SW27 to SW28, SW28 to SW29, SW29 to SW30, SW30 to SW31
Connections:
- net +BATT: now also J3.4 (Pin_4), J3.5 (Pin_5)
- net GND: now also J3.27 (Pin_27), R4.1; no longer R9.2
- net LCD_RST: now also U1.9 (PC1); no longer U1.5 (PH0)
- net NCS: now also U1.33 (PB12); no longer U1.6 (PH1)
- net RD: no longer J3.5 (Pin_5)
- net WR: no longer J3.4 (Pin_4)
- net at J3.25 (Pin_25), R9.1: now also R3.1; no longer R8.2
- net at J3.22 (Pin_22): now also R5.2, R4.2
- net at J3.23 (Pin_23), R6.2: now also R5.1
- net at J3.24 (Pin_24): now also R8.1, R9.2; no longer R5.2
- net C86: no longer names the net of U1.21 (PA5)
- net C86: no longer J3.27 (Pin_27)
- new net: R7.1, R8.2
- new net: R6.1, R7.2
- new net: J3.26 (Pin_26), R3.2
- no-connect marks 30 -> 28
Other:
- moved on the sheet: R8

Commit message: Update.
Parts:
- removed J2: Conn_01x04, Connector_PinHeader_2.54mm:PinHeader_1x04_P2.54mm_Vertical, symbol Connector_Generic:Conn_01x04
- removed R3, R4, R5, R6, R7, R8, R9: 1K, Resistor_SMD:R_0603_1608Metric_Pad0.98x0.95mm_HandSolder, symbol Device:R_US
- removed U1: STM32L071RZTx, Package_QFP:LQFP-64_10x10mm_P0.5mm, symbol MCU_ST_STM32L0:STM32L071RZTx
- added C13, C14, C7, C8, C9: C, Capacitor_SMD:C_0603_1608Metric_Pad1.08x0.95mm_HandSolder, symbol Device:C
- added TP1, TP10, TP11, TP12, TP13, TP16, TP18, TP19, TP2, TP20, TP21, TP3, TP4, TP5, TP6, TP7, TP8, TP9: TestPoint, TestPoint:TestPoint_THTPad_1.0x1.0mm_Drill0.5mm, symbol Connector:TestPoint
- added TP14, TP15, TP17, TP22: TestPoint, TestPoint:TestPoint_THTPad_2.0x2.0mm_Drill1.0mm, symbol Connector:TestPoint
- added U1: STM32F407VGTx, Package_QFP:LQFP-100_14x14mm_P0.5mm, symbol MCU_ST_STM32F4:STM32F407VGTx
- R2: renamed from R1; value R_US -> 10k; now in the parts list
- renumbered C7 to C10, C8 to C11, C9 to C12, C10 to C15, J3 to J2, R2 to R1, SW22 to SW21, SW23 to SW22, SW24 to SW23, SW25 to SW24, SW26 to SW25, SW27 to SW26, SW28 to SW27, SW29 to SW28, SW30 to SW29, SW31 to SW30, SW21 to SW31
Connections:
- net +BATT: now also TP1.1, U1.100 (VDD), U1.11 (VDD), U1.19 (VDD), U1.21 (VREF+), U1.22 (VDDA), U1.28 (VDD), U1.50 (VDD), U1.6 (VBAT), U1.75 (VDD)
- net A0: now also TP2.1, U1.7 (PC13)
- net GND: now also C13.2, C14.2, C7.2, C8.2, C9.2, TP22.1, TP3.1, U1.10 (VSS), U1.20 (VSSA), U1.27 (VSS), U1.74 (VSS), U1.99 (VSS)
- net LCD_RST: now also TP5.1, U1.16 (PC1)
- net NCS: now also TP6.1, U1.51 (PB12)
- net NRST: now also TP14.1, U1.14 (NRST)
- net SCL: now also TP8.1, U1.47 (PB10)
- net SI: now also TP4.1, U1.18 (PC3)
- net SWCLK: now also TP17.1, U1.76 (PA14)
- net SWDIO: now also TP15.1, U1.72 (PA13)
- net X1: now also TP21.1, U1.35 (PB0)
- net X2: now also TP20.1, U1.36 (PB1)
- net X3: now also TP19.1, U1.37 (PB2)
- net X4: now also TP18.1, U1.89 (PB3)
- net X5: now also TP16.1, U1.90 (PB4)
- net X6: now also TP13.1, U1.91 (PB5)
- net Y1: now also TP12.1, U1.92 (PB6)
- net Y2: now also TP11.1, U1.93 (PB7)
- net Y3: now also TP10.1, U1.95 (PB8)
- net Y4: now also TP9.1, U1.96 (PB9)
- net Y5: now also TP7.1, U1.48 (PB11)
- net at J2.25 (Pin_25): now also C13.1
- net at J2.24 (Pin_24): now also C8.1
- net at J2.23 (Pin_23): now also C14.1
- net at J2.22 (Pin_22): now also C7.1
- net at J2.26 (Pin_26): now also C9.1
- net at R1.1: now also U1.94 (BOOT0)
- no-connect marks 28 -> 0
Other:
- moved on the sheet: C1, R1, R2, SW31
