File: 01_EDA/KS100.kicad_pcb (KiCad board)
At the start: 2 copper layers, 80 x 80 mm, 55 parts, among them J1 Conn_01x02_Pin, J2 Conn_01x04, J3 DEM 128064E1 FGH, SW1 SW_Push, SW10 SW_Push, SW11 SW_Push, SW12 SW_Push, SW13 SW_Push, SW14 SW_Push, SW15 SW_Push, SW16 SW_Push, SW17 SW_Push, SW18 SW_Push, SW19 SW_Push, SW2 SW_Push, SW20 SW_Push, SW21 SW_Push, SW22 SW_Push, SW23 SW_Push, SW24 SW_Push, SW25 SW_Push, SW26 SW_Push, SW27 SW_Push, SW28 SW_Push, SW29 SW_Push, SW3 SW_Push, SW30 SW_Push, SW31 SW_Push, SW4 SW_Push, SW5 SW_Push, SW6 SW_Push, SW7 SW_Push, SW8 SW_Push, SW9 SW_Push, U1 STM32L071RZTx

Commit message: Update.
Parts:
- removed C1: C, Capacitor_SMD:C_0603_1608Metric_Pad1.08x0.95mm_HandSolder
- removed SW31: SW_Push, Button_Switch_THT:SW_PUSH_1P1T_6x3.5mm_H4.3_APEM_MJTP1243
- added ?: , , F.Cu at (190.0, 69.0)
- added ?: , , F.Cu at (190.0, 145.0)
- added ?: , , F.Cu at (114.0, 145.0)
- added REF**: MountingHole_3mm, MountingHole:MountingHole_3mm, F.Cu at (115.0, 70.0)
- J1: footprint Connector_PinHeader_2.00mm:PinHeader_1x02_P2.00mm_Vertical -> Connector_JST:JST_VH_B2P-VH-B_1x02_P3.96mm_Vertical
- moved J1 2.93 mm to (115.7, 100.0), turned to 90 degrees
Routing:
- net GND: track 41.8 -> 48.2 mm
- net +BATT: track 37.9 -> 41.5 mm
- net /Calculator/SCL: track 133.0 -> 133.9 mm
- net /Calculator/LCD_RST: track 32.1 -> 32.9 mm
- net /Calculator/Y5: track 108.1 -> 108.7 mm
- net /Calculator/WR: track 32.3 -> 32.8 mm
Other:
- board size 80 x 80 mm -> 82 x 82 mm

Commit message: Update.
Parts:
- removed ? (x3): , 
- removed the J2 at (149.7, 109.1)
- removed R10, R11, R12, R5, R6, R7, R8, R9: R_US, Resistor_SMD:R_0603_1608Metric_Pad0.98x0.95mm_HandSolder
- removed REF**: MountingHole_3mm, MountingHole:MountingHole_3mm
- added C1: C, Capacitor_SMD:C_0603_1608Metric_Pad1.08x0.95mm_HandSolder, F.Cu at (149.9, 80.3)
- added C13: C, Capacitor_SMD:C_0603_1608Metric_Pad1.08x0.95mm_HandSolder, F.Cu at (132.7, 77.2)
- added C14: C, Capacitor_SMD:C_0603_1608Metric_Pad1.08x0.95mm_HandSolder, F.Cu at (135.7, 77.2)
- added C7: C, Capacitor_SMD:C_0603_1608Metric_Pad1.08x0.95mm_HandSolder, F.Cu at (137.2, 77.2)
- added C8: C, Capacitor_SMD:C_0603_1608Metric_Pad1.08x0.95mm_HandSolder, F.Cu at (134.2, 77.2)
- added C9: C, Capacitor_SMD:C_0603_1608Metric_Pad1.08x0.95mm_HandSolder, F.Cu at (131.2, 77.2)
- added SW31: SW_Push, Button_Switch_THT:SW_PUSH_1P1T_6x3.5mm_H4.3_APEM_MJTP1243, F.Cu at (158.3, 78.0)
- added TP1: TestPoint, TestPoint:TestPoint_THTPad_1.0x1.0mm_Drill0.5mm, F.Cu at (115.8, 106.6)
- added TP10: TestPoint, TestPoint:TestPoint_THTPad_1.0x1.0mm_Drill0.5mm, F.Cu at (180.6, 123.8)
- added TP11: TestPoint, TestPoint:TestPoint_THTPad_1.0x1.0mm_Drill0.5mm, F.Cu at (179.8, 118.0)
- added TP12: TestPoint, TestPoint:TestPoint_THTPad_1.0x1.0mm_Drill0.5mm, F.Cu at (176.2, 109.0)
- added TP13: TestPoint, TestPoint:TestPoint_THTPad_1.0x1.0mm_Drill0.5mm, F.Cu at (171.4, 107.0)
- added TP14: TestPoint, TestPoint:TestPoint_THTPad_2.0x2.0mm_Drill1.0mm, F.Cu at (170.2, 86.0)
- added TP15: TestPoint, TestPoint:TestPoint_THTPad_2.0x2.0mm_Drill1.0mm, F.Cu at (170.2, 89.2)
- added TP16: TestPoint, TestPoint:TestPoint_THTPad_1.0x1.0mm_Drill0.5mm, F.Cu at (161.3, 105.9)
- added TP17: TestPoint, TestPoint:TestPoint_THTPad_2.0x2.0mm_Drill1.0mm, F.Cu at (170.2, 92.4)
- added TP18: TestPoint, TestPoint:TestPoint_THTPad_1.0x1.0mm_Drill0.5mm, F.Cu at (151.2, 124.0)
- added TP19: TestPoint, TestPoint:TestPoint_THTPad_1.0x1.0mm_Drill0.5mm, F.Cu at (141.0, 117.0)
- added TP2: TestPoint, TestPoint:TestPoint_THTPad_1.0x1.0mm_Drill0.5mm, F.Cu at (162.6, 68.8)
- added TP20: TestPoint, TestPoint:TestPoint_THTPad_1.0x1.0mm_Drill0.5mm, F.Cu at (130.8, 117.2)
- added TP21: TestPoint, TestPoint:TestPoint_THTPad_1.0x1.0mm_Drill0.5mm, F.Cu at (120.0, 116.8)
- added TP22: TestPoint, TestPoint:TestPoint_THTPad_2.0x2.0mm_Drill1.0mm, F.Cu at (170.2, 95.4)
- added TP3: TestPoint, TestPoint:TestPoint_THTPad_1.0x1.0mm_Drill0.5mm, F.Cu at (115.8, 90.8)
- added TP4: TestPoint, TestPoint:TestPoint_THTPad_1.0x1.0mm_Drill0.5mm, F.Cu at (149.8, 68.6)
- added TP5: TestPoint, TestPoint:TestPoint_THTPad_1.0x1.0mm_Drill0.5mm, F.Cu at (163.8, 71.2)
- added TP6: TestPoint, TestPoint:TestPoint_THTPad_1.0x1.0mm_Drill0.5mm, F.Cu at (165.0, 68.8)
- added TP7: TestPoint, TestPoint:TestPoint_THTPad_1.0x1.0mm_Drill0.5mm, F.Cu at (145.2, 131.4)
- added TP8: TestPoint, TestPoint:TestPoint_THTPad_1.0x1.0mm_Drill0.5mm, F.Cu at (152.8, 71.0)
- added TP9: TestPoint, TestPoint:TestPoint_THTPad_1.0x1.0mm_Drill0.5mm, F.Cu at (181.7, 129.1)
- R2: renamed from R1; value R_US -> 10k
- U1: value STM32L071RZTx -> STM32F407VGTx; footprint Package_QFP:LQFP-64_10x10mm_P0.5mm -> Package_QFP:LQFP-100_14x14mm_P0.5mm
- moved C3 24.3 mm to (144.7, 82.6), turned to 90 degrees
- moved C4 17.6 mm to (138.8, 100.5)
- moved C6 17.1 mm to (150.7, 83.4), turned to 0 degrees
- moved C2 15.6 mm to (155.0, 103.4), turned to 180 degrees
- moved C5 11.5 mm to (153.2, 82.5), turned to 90 degrees
- moved R1 7.46 mm to (160.1, 90.0)
- moved U1 5.74 mm to (149.3, 93.1)
- moved R2 5.48 mm to (149.9, 81.8)
- moved C15 0.74 mm to (147.1, 77.0), turned to -90 degrees
- renumbered C8 to C10, C9 to C11, C10 to C12, C7 to C15, J3 to J2, R2 to R1
Connections:
- J2 pad 27: /Calculator/C86 -> GND
- J2 pad 4: /Calculator/WR -> +BATT
- J2 pad 5: /Calculator/RD -> +BATT
- U1 pad 1: +BATT -> unconnected-(U1-PE2-Pad1)
- U1 pad 10: unconnected-(U1-PC2-Pad10) -> GND
- U1 pad 11: /Calculator/SI -> +BATT
- U1 pad 12: GND -> unconnected-(U1-PH0-Pad12)
- U1 pad 13: +BATT -> unconnected-(U1-PH1-Pad13)
- U1 pad 14: unconnected-(U1-PA0-Pad14) -> /Calculator/NRST
- U1 pad 16: unconnected-(U1-PA2-Pad16) -> /Calculator/LCD_RST
- U1 pad 18: GND -> /Calculator/SI
- U1 pad 2: /Calculator/A0 -> unconnected-(U1-PE3-Pad2)
- U1 pad 20: unconnected-(U1-PA4-Pad20) -> GND
- U1 pad 21: /Calculator/C86 -> +BATT
- U1 pad 22: unconnected-(U1-PA6-Pad22) -> +BATT
- U1 pad 26: /Calculator/X1 -> unconnected-(U1-PA3-Pad26)
- U1 pad 27: /Calculator/X2 -> GND
- U1 pad 28: /Calculator/X3 -> +BATT
- U1 pad 29: /Calculator/SCL -> unconnected-(U1-PA4-Pad29)
- U1 pad 3: /Calculator/WR -> unconnected-(U1-PE4-Pad3)
- U1 pad 30: /Calculator/Y5 -> unconnected-(U1-PA5-Pad30)
- U1 pad 31: GND -> unconnected-(U1-PA6-Pad31)
- U1 pad 32: +BATT -> unconnected-(U1-PA7-Pad32)
- U1 pad 35: unconnected-(U1-PB14-Pad35) -> /Calculator/X1
- U1 pad 36: unconnected-(U1-PB15-Pad36) -> /Calculator/X2
- U1 pad 37: unconnected-(U1-PC6-Pad37) -> /Calculator/X3
- U1 pad 4: /Calculator/RD -> unconnected-(U1-PE5-Pad4)
- U1 pad 46: /Calculator/SWDIO -> unconnected-(U1-PE15-Pad46)
- U1 pad 47: GND -> /Calculator/SCL
- U1 pad 48: +BATT -> /Calculator/Y5
- U1 pad 49: /Calculator/SWCLK -> unconnected-(U1-VCAP_1-Pad49)
- U1 pad 5: /Calculator/LCD_RST -> unconnected-(U1-PE6-Pad5)
- U1 pad 50: unconnected-(U1-PA15-Pad50) -> +BATT
- U1 pad 51: unconnected-(U1-PC10-Pad51) -> /Calculator/NCS
- U1 pad 55: /Calculator/X4 -> unconnected-(U1-PD8-Pad55)
- U1 pad 56: /Calculator/X5 -> unconnected-(U1-PD9-Pad56)
- U1 pad 57: /Calculator/X6 -> unconnected-(U1-PD10-Pad57)
- U1 pad 58: /Calculator/Y1 -> unconnected-(U1-PD11-Pad58)
- U1 pad 59: /Calculator/Y2 -> unconnected-(U1-PD12-Pad59)
- U1 pad 6: /Calculator/NCS -> +BATT
- U1 pad 60: Net-(U1-BOOT0) -> unconnected-(U1-PD13-Pad60)
- U1 pad 61: /Calculator/Y3 -> unconnected-(U1-PD14-Pad61)
- U1 pad 62: /Calculator/Y4 -> unconnected-(U1-PD15-Pad62)
- U1 pad 63: GND -> unconnected-(U1-PC6-Pad63)
- U1 pad 64: +BATT -> unconnected-(U1-PC7-Pad64)
- U1 pad 7: /Calculator/NRST -> /Calculator/A0
Routing:
- net /Calculator/SCL: track 133.9 -> 52.8 mm, vias 1 -> 2
- net /Calculator/RD: track 35.0 -> 0.00 mm, vias 2 -> 0
- net /Calculator/C86: track 33.1 -> 0.00 mm, vias 2 -> 0
- net /Calculator/WR: track 32.8 -> 0.00 mm, vias 2 -> 0
- net +BATT: track 41.5 -> 10.5 mm, vias 0 -> 2
- net /Calculator/SWDIO: track 8.89 -> 36.3 mm, vias 0 -> 2
- net GND: track 48.2 -> 29.1 mm, vias 8 -> 16
- net Net-(J2-Pin_26): track 14.2 -> 3.64 mm
- net /Calculator/X4: track 48.0 -> 58.0 mm
- net /Calculator/LCD_RST: track 32.9 -> 42.5 mm
- net /Calculator/NCS: track 42.0 -> 51.0 mm
- net Net-(J2-Pin_23): track 11.8 -> 3.35 mm
- net /Calculator/X3: track 48.9 -> 56.0 mm
- net Net-(J2-Pin_22): track 10.2 -> 3.26 mm
- net Net-(J2-Pin_24): track 9.63 -> 3.45 mm
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Other:
- board text added: "BAT"
- board text added: "GND"
- board text added: "KS100 R1.0"
- board text added: "NRST"
- board text added: "SWCLK"
- board text added: "SWDIO"
